File: eagle/bahilizator.kicad_pcb (KiCad board)
At the start: 2 copper layers, 60 parts

Commit message: hw: BC547 footprint changed TO-92 → SOT-23
- All 8× BC547 NPN transistors now SMD (SOT-23)
- Package_TO_SOT_SMD:SOT-23 footprint in KiCad library
- Regenerated bahilizator.kicad_pcb
Parts:
- removed the Q_HOPA at (60.0, 55.0)
- removed the Q_HOPB at (65.0, 55.0)
- removed the Q_PWRKEY at (10.0, 55.0)
- added Q_HOPA: , Package_TO_SOT_SMD:SOT-23, F.Cu at (60.0, 55.0)
- added Q_HOPB: , Package_TO_SOT_SMD:SOT-23, F.Cu at (65.0, 55.0)
- added Q_PWRKEY: , Package_TO_SOT_SMD:SOT-23, F.Cu at (10.0, 55.0)
- Q_COIN1, Q_COIN2, Q_COIN3, Q_COIN4, Q_COIN5, Q_COIN6: footprint Package_TO_SOT_THT:TO-92_Inline_Wide -> Package_TO_SOT_SMD:SOT-23
Changed lines of the file:
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@@
     )
   )
-  (footprint "Package_TO_SOT_THT:TO-92_Inline_Wide" (layer "F.Cu")
+  (footprint "Package_TO_SOT_SMD:SOT-23" (layer "F.Cu")
     (at 25 55) (rotation 0)
     (attr through_hole)
@@
     )
   )
-  (footprint "Package_TO_SOT_THT:TO-92_Inline_Wide" (layer "F.Cu")
+  (footprint "Package_TO_SOT_SMD:SOT-23" (layer "F.Cu")
     (at 30 55) (rotation 0)
     (attr through_hole)
@@
     )
   )
-  (footprint "Package_TO_SOT_THT:TO-92_Inline_Wide" (layer "F.Cu")
+  (footprint "Package_TO_SOT_SMD:SOT-23" (layer "F.Cu")
     (at 35 55) (rotation 0)
     (attr through_hole)
@@
     )
   )
-  (footprint "Package_TO_SOT_THT:TO-92_Inline_Wide" (layer "F.Cu")
+  (footprint "Package_TO_SOT_SMD:SOT-23" (layer "F.Cu")
     (at 40 55) (rotation 0)
     (attr through_hole)
@@
     )
   )
-  (footprint "Package_TO_SOT_THT:TO-92_Inline_Wide" (layer "F.Cu")
+  (footprint "Package_TO_SOT_SMD:SOT-23" (layer "F.Cu")
     (at 45 55) (rotation 0)
     (attr through_hole)
@@
     )
   )
-  (footprint "Package_TO_SOT_THT:TO-92_Inline_Wide" (layer "F.Cu")
+  (footprint "Package_TO_SOT_SMD:SOT-23" (layer "F.Cu")
     (at 50 55) (rotation 0)
     (attr through_hole)
@@
     )
   )
-  (footprint "Package_TO_SOT_THT:TO-92_Inline_Wide" (layer "F.Cu")
+  (footprint "Package_TO_SOT_SMD:SOT-23" (layer "F.Cu")
     (at 60 55) (rotation 0)
     (attr through_hole)
@@
     )
   )
-  (footprint "Package_TO_SOT_THT:TO-92_Inline_Wide" (layer "F.Cu")
+  (footprint "Package_TO_SOT_SMD:SOT-23" (layer "F.Cu")
     (at 65 55) (rotation 0)
     (attr through_hole)
@@
     )
   )
-  (footprint "Package_TO_SOT_THT:TO-92_Inline_Wide" (layer "F.Cu")
+  (footprint "Package_TO_SOT_SMD:SOT-23" (layer "F.Cu")
     (at 10 55) (rotation 0)
     (attr through_hole)

Commit message: hw: PCF8574P footprint changed DIP-16 → SOIC-16
- Package_SO:SOIC-16_3.9x9.9mm_P1.27mm (SMD)
- All components now SMD except connectors and crystal
- Regenerated bahilizator.kicad_pcb
Parts:
- U2: footprint Package_DIP:DIP-16_W7.62mm -> Package_SO:SOIC-16_3.9x9.9mm_P1.27mm
Changed lines of the file:
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@@
     )
   )
-  (footprint "Package_DIP:DIP-16_W7.62mm" (layer "F.Cu")
+  (footprint "Package_SO:SOIC-16_3.9x9.9mm_P1.27mm" (layer "F.Cu")
     (at 80 10) (rotation 0)
     (attr through_hole)

Commit message: fix: KiCad PCB format — (net) at top level, no (nets) wrapper
- KiCad PCB uses individual (net N "name") at root level
- (nets ...) wrapper only valid in netlist format, not PCB
- Regenerated bahilizator.kicad_pcb — should parse without errors
Other:
- board text added: "STM32F103C8T6"
- board text removed: "STM32F103C8T6 Bluepill"
