File: eagle/bahilizator.kicad_sch (KiCad schematic)
At the start: 58 parts, among them J1 SWD, J2 SIM800L, J3 NRI_G13, Q1 BC547, Q2 BC547, Q3 BC547, Q4 BC547, Q5 BC547, Q6 BC547, Q7 BC547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

Commit message: fix: KiCad schematic loads successfully — 5019 lines, ERC passes
- Fixed missing '(' before pin definitions in lib_symbols
- Pin format: (pin type line (at x y rot) (length N) (name ...) (number ...))
- 17 symbol definitions, 63 instances, 5 power flags
- ERC: 250 violations (unconnected pins — expected, wiring not done yet)
- kicad-cli sch erc passes without parse errors
Parts:
- removed D1: RED, symbol LED_THT:LED
- removed D2: GREEN, symbol LED_THT:LED
- added D1: RED, symbol Device:LED
- added D2: GREEN, symbol Device:LED
Connections:
- new net: D2.1 (A), R31.2
- new net: D1.1 (A), R30.2
- new net: Q8.1 (B), U1.24 (VDD)
- new net: U2.11 (P7), U3.5 (SDA)
- new net: Q6.3 (C), U1.6 (PD1)
- new net: Q7.1 (B), U1.7 (NRST)
- new net: Q6.2 (E), U1.8 (VSSA)
Other:
- title: Бахилизатор v2.0 — STM32F103C8T6 Bluepill -> Bahilizator v2.0 - STM32F103C8T6 Bluepill
